File: KiCAD/enc28j60_buffered_tht_shield/enc28j60_buffered_tht_shield.kicad_pcb (KiCad board)
At the start: 2 copper layers, 68.6 x 53.3 mm, 41 parts, among them J1 AVR-ISP-6, J2 RJ45_MagJack_LMJTAB881X43M-L, J3 Conn_01x05_Male, J4 Conn_01x03_Male, P1 CONN_01X01, P2 CONN_01X01, P3 CONN_01X01, P4 CONN_01X01, P5 Digital, P6 Power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

Commit message: Fix library problem.
Parts:
- moved C12 0.85 mm to (128.9, 119.5), turned to 270 degrees
- moved C11 0.59 mm to (125.9, 116.6)
- moved C13 0.07 mm to (134.8, 123.3)
Routing:
- net +3V3: track 135.8 -> 133.4 mm
